File: src/PT Hub/PT Hub.kicad_sch (KiCad schematic)
At the start: 18 parts

Commit message: sc
shcematic
Parts:
- gave numbers to parts that had none: 18

Commit message: 1 symbol
Parts:
- removed C1: 1uF, PT-Hub:CAP_0603, symbol PT-Hub:CAP_0603
- removed C2: 1uF, symbol PT-Hub:CAP_0603
- removed D1: SML-LX1206GC-TR, symbol PT-Hub:SML-LX1206GC-TR
- removed H1, H2, H3, H4: Mounting-Hole, symbol PT-Hub:Mounting-Hole
- removed LOGO1: Logo, symbol PT-Hub:Logo
- removed P1: 20021511-00026T4LF, PT-Hub:20021511-00026T4LF, symbol PT-Hub:20021511-00026T4LF
- removed P2, P3, P5, P6, P7, P8, P9: 39299043, CONN_4840.2201_SCH, symbol PT-Hub:39299043
- removed P4: 39299043, symbol PT-Hub:39299043
- removed R1: 750, symbol PT-Hub:RES_0603
- added P?: 20021511-00026T4LF, CONN20_D10-RA-BK_SUL, symbol PT-Hub:20021511-00026T4LF
Other:
- note removed: "Capacitor"
- note removed: "LED"
- note removed: "Micellaneous"
- note removed: "PT Connectors"
- note removed: "Pressure Transducer Connectors"

Commit message: copy paste again
Parts:
- removed P?: 20021511-00026T4LF, CONN20_D10-RA-BK_SUL, symbol PT-Hub:20021511-00026T4LF
- added C?: 1uF, PT-Hub:CAP_0603, symbol PT-Hub:CAP_0603
- added C?: 1uF, symbol PT-Hub:CAP_0603
- added D?: SML-LX1206GC-TR, symbol PT-Hub:SML-LX1206GC-TR
- added H? (x4): Mounting-Hole, symbol PT-Hub:Mounting-Hole
- added LOGO?: Logo, symbol PT-Hub:Logo
- added P? (x7): 39299043, CONN_4840.2201_SCH, symbol PT-Hub:39299043
- added P?: 39299043, symbol PT-Hub:39299043
- added P?: 20021511-00026T4LF, PT-Hub:20021511-00026T4LF, symbol PT-Hub:20021511-00026T4LF
- added R?: 750, symbol PT-Hub:RES_0603
Connections:
- new net: D?.1, R?.2
- new net 5V: C?.1, C?.1, D?.2, P?.1, P?.1 (+12V), P?.1 (+12V), P?.1 (+12V), P?.1 (+12V), P?.1 (+12V), P?.1 (+12V), P?.1 (+12V), P?.1 (+12V), P?.2, P?.3, P?.4
- new net Earth: C?.2, C?.2, P?.21, P?.22, P?.23, P?.24, P?.25, P?.26, P?.4, P?.4, P?.4, P?.4, P?.4, P?.4, P?.4, P?.4, R?.1
- new net PT1+: P?.2 (GND), P?.5
- new net PT1-: P?.3, P?.6
- new net PT2+: P?.2 (GND), P?.7
- new net PT2-: P?.3, P?.8
- new net PT3+: P?.2 (GND), P?.9
- new net PT3-: P?.10, P?.3
- new net PT4+: P?.11, P?.2 (GND)
- new net PT4-: P?.12, P?.3
- new net PT5+: P?.13, P?.2 (GND)
- new net PT5-: P?.14, P?.3
- new net PT6+: P?.15, P?.2 (GND)
- new net PT6-: P?.16, P?.3
- new net PT7+: P?.17, P?.2 (GND)
- new net PT7-: P?.18, P?.3
- new net PT8+: P?.19, P?.2 (GND)
- new net PT8-: P?.20, P?.3
Other:
- note added: "Capacitor"
- note added: "LED"
- note added: "Micellaneous"
- note added: "PT Connectors"
- note added: "Pressure Transducer Connectors"

Commit message: footprints and PDB editor started
Parts:
- C2: renamed from C?; footprint (none) -> PT-Hub:CAP_0603
- D1: renamed from D?; footprint (none) -> PT-Hub:SML-LX1206GC-TR
- H1, H2, H3, H4: renamed from H?; footprint (none) -> PT-Hub:MountingHole_4.3mm_M4_DIN965
- LOGO1: renamed from LOGO?; footprint (none) -> PT-Hub:Logo
- P2, P3, P5, P6, P7, P8, P9: renamed from P?; footprint CONN_4840.2201_SCH -> PT-Hub:39299043
- P4: renamed from P?; footprint (none) -> PT-Hub:39299043
- R1: renamed from R?; footprint (none) -> PT-Hub:RES_0603
- gave numbers to parts that had none: 2
Other:
- note added: "Power Supply Decoupling"
- note removed: "Capacitor"
- company: (none) -> Sun Devil Rocketry
- title: (none) -> PT-Hub

Commit message: modified PT hub to be usable with hybrids PTs
Connections:
- net PT5- is gone; now on net Earth: P1.14, P2.3
- net PT6- is gone; now on net Earth: P1.16, P6.3
- net PT7- is gone; now on net Earth: P1.18, P3.3
- net PT8- is gone; now on net Earth: P1.20, P9.3
- net 5V: no longer P1.3, P1.4, P2.1 (+12V), P3.1 (+12V), P6.1 (+12V), P9.1 (+12V)
- new net VIN: P1.3, P1.4, P2.1 (+12V), P3.1 (+12V), P6.1 (+12V), P9.1 (+12V)
Other:
- note added: "Engine Pressure"
- note added: "Extra"
- note added: "Fuel Flow High Pressure"
- note added: "Fuel Flow Low Pressure"
- note added: "Fuel Pressure"
- note added: "LOX Flow High Pressure"
- note added: "LOX Flow Low Pressure"
- note added: "LOX Pressure"
